File: Motor Control.kicad_pcb (KiCad board)
At the start: 2 copper layers, 160 x 100 mm, 103 parts, among them J1 Conn_01x05_Pin, J2 Conn_01x06_Pin, J3 USB_B, J4 Conn_01x02_Socket, J5 Conn_01x02_Socket, J6 Conn_01x02_Socket, Q10 IRLZ44N, Q11 IRLZ44N, Q110 IRLZ44N, Q111 BC557, Q112 BC547, Q113 BC557, Q12 BC547, Q13 BC557, Q14 BC547, Q15 BC557, Q16 BC557, Q17 BC547, Q18 BC547, Q2 BC547, Q210 BC547, Q6 BC547, Q7 BC557, Q9 IRLZ44N, SW1 RotaryEncoder_Switch_MP, U10 LM317_TO-220, U110 4N35, U2 4N35, U3 PIC18F26K22-xSP, U4 MCP2221AxP, U5 L78L05_TO92, U6 4N35, U7 4N35, U8 HCPL7510, U9 74AHC595

Commit message: Placement H bridge & PSU
Parts:
- removed C11, C4, C8: 100nF, Capacitor_THT:C_Rect_L7.2mm_W2.5mm_P5.00mm_FKS2_FKP2_MKS2_MKP2
- removed C12: 150pF, Capacitor_THT:C_Rect_L7.2mm_W2.5mm_P5.00mm_FKS2_FKP2_MKS2_MKP2
- removed C14: 330uF, Capacitor_THT:CP_Radial_D8.0mm_P5.00mm
- removed C15, C16: 1uF, Capacitor_THT:CP_Radial_D5.0mm_P2.50mm
- removed C6: 1uF, Capacitor_THT:CP_Radial_D4.0mm_P2.00mm
- removed C9: 10nF, Capacitor_THT:C_Rect_L7.2mm_W2.5mm_P5.00mm_FKS2_FKP2_MKS2_MKP2
- removed D2, D3, D4: 1N4148, Diode_THT:D_DO-35_SOD27_P7.62mm_Horizontal
- removed Q10, Q11, Q9: IRLZ44N, Package_TO_SOT_THT:TO-220-3_Horizontal_TabDown
- removed Q12, Q14, Q17, Q18, Q2, Q6: BC547, Package_TO_SOT_THT:TO-92_Inline_Wide
- removed Q13, Q15, Q16, Q7: BC557, Package_TO_SOT_THT:TO-92_Inline_Wide
- removed R10, R30: 270k, Resistor_THT:R_Axial_DIN0207_L6.3mm_D2.5mm_P10.16mm_Horizontal
- removed R13, R2, R25, R26, R28, R38, R40: 1k, Resistor_THT:R_Axial_DIN0207_L6.3mm_D2.5mm_P10.16mm_Horizontal
- removed R15, R22, R24: 150, Resistor_THT:R_Axial_DIN0207_L6.3mm_D2.5mm_P10.16mm_Horizontal
- removed R17, R20, R21: 10R, Resistor_THT:R_Axial_DIN0207_L6.3mm_D2.5mm_P10.16mm_Horizontal
- removed R18: 0R20, Resistor_THT:R_Axial_DIN0516_L15.5mm_D5.0mm_P20.32mm_Horizontal
- removed R31: 47k, Resistor_THT:R_Axial_DIN0207_L6.3mm_D2.5mm_P10.16mm_Horizontal
- removed R33: 68R, Resistor_THT:R_Axial_DIN0207_L6.3mm_D2.5mm_P10.16mm_Horizontal
- removed R34, R35, R8: 180, Resistor_THT:R_Axial_DIN0207_L6.3mm_D2.5mm_P10.16mm_Horizontal
- removed R36, R37, R6: 10k, Resistor_THT:R_Axial_DIN0207_L6.3mm_D2.5mm_P10.16mm_Horizontal
- removed R44: 3k3, Resistor_THT:R_Axial_DIN0207_L6.3mm_D2.5mm_P10.16mm_Horizontal
- removed R45: 390, Resistor_THT:R_Axial_DIN0207_L6.3mm_D2.5mm_P10.16mm_Horizontal
- removed U10: LM317_TO-220, Package_TO_SOT_THT:TO-220-3_Horizontal_TabDown
- removed U2, U6, U7: 4N35, Package_DIP:DIP-6_W7.62mm_Socket_LongPads
- removed U5: L78L05_TO92, Package_TO_SOT_THT:TO-92_Inline_Wide
- removed U8: HCPL7510, Package_DIP:DIP-8_W7.62mm_Socket_LongPads
- added C120: 1uF, Capacitor_THT:CP_Radial_D4.0mm_P2.00mm, F.Cu at (348.6, 129.8)
- added C900: 330uF, Capacitor_THT:CP_Radial_D8.0mm_P5.00mm, F.Cu at (389.9, 48.3)
- added C901: 1uF, Capacitor_THT:CP_Radial_D5.0mm_P2.50mm, F.Cu at (359.4, 55.9)
- added C902: 1uF, Capacitor_THT:CP_Radial_D5.0mm_P2.50mm, F.Cu at (359.4, 62.2)
- added C903: 100nF, Capacitor_THT:C_Rect_L7.2mm_W2.5mm_P5.00mm_FKS2_FKP2_MKS2_MKP2, F.Cu at (345.4, 53.3)
- added C904: 100nF, Capacitor_THT:C_Rect_L7.2mm_W2.5mm_P5.00mm_FKS2_FKP2_MKS2_MKP2, F.Cu at (349.2, 66.6)
- added C905: 10nF, Capacitor_THT:C_Rect_L7.2mm_W2.5mm_P5.00mm_FKS2_FKP2_MKS2_MKP2, F.Cu at (345.4, 66.7)
- added C906: 100nF, Capacitor_THT:C_Rect_L7.2mm_W2.5mm_P5.00mm_FKS2_FKP2_MKS2_MKP2, F.Cu at (329.6, 64.1)
- added C907: 100nF, Capacitor_THT:C_Rect_L7.2mm_W2.5mm_P5.00mm_FKS2_FKP2_MKS2_MKP2, F.Cu at (326.4, 64.1)
- added D120: 1N4148, Diode_THT:D_DO-35_SOD27_P7.62mm_Horizontal, F.Cu at (353.1, 124.5)
- added D900: 1N4148, Diode_THT:D_DO-35_SOD27_P7.62mm_Horizontal, F.Cu at (370.8, 62.2)
- added D901: 1N4148, Diode_THT:D_DO-35_SOD27_P7.62mm_Horizontal, F.Cu at (370.8, 59.1)
- added Q120: IRLZ44N, Package_TO_SOT_THT:TO-220-3_Horizontal_TabDown, F.Cu at (375.9, 119.4)
- added Q121: BC557, Package_TO_SOT_THT:TO-92_Inline_Wide, F.Cu at (345.4, 119.4)
- added Q122: BC547, Package_TO_SOT_THT:TO-92_Inline_Wide, F.Cu at (353.1, 119.4)
- added Q123: BC557, Package_TO_SOT_THT:TO-92_Inline_Wide, F.Cu at (353.1, 129.5)
- added Q130: IRLZ44N, Package_TO_SOT_THT:TO-220-3_Horizontal_TabDown, F.Cu at (375.9, 99.1)
- added Q131: BC547, Package_TO_SOT_THT:TO-92_Inline_Wide, F.Cu at (353.1, 99.1)
- added Q132: BC557, Package_TO_SOT_THT:TO-92_Inline_Wide, F.Cu at (353.1, 107.3)
- added Q140: IRLZ44N, Package_TO_SOT_THT:TO-220-3_Horizontal_TabDown, F.Cu at (375.9, 81.3)
- added Q141: BC547, Package_TO_SOT_THT:TO-92_Inline_Wide, F.Cu at (353.1, 81.3)
- added Q142: BC557, Package_TO_SOT_THT:TO-92_Inline_Wide, F.Cu at (353.1, 89.5)
- added Q220: BC547, Package_TO_SOT_THT:TO-92_Inline_Wide, F.Cu at (324.5, 123.2)
- added Q230: BC547, Package_TO_SOT_THT:TO-92_Inline_Wide, F.Cu at (324.5, 100.3)
- added Q240: BC547, Package_TO_SOT_THT:TO-92_Inline_Wide, F.Cu at (324.5, 82.5)
- added R000: 0R20, Resistor_THT:R_Axial_DIN0516_L15.5mm_D5.0mm_P20.32mm_Horizontal, F.Cu at (355.6, 68.6)
- added R120: 10R, Resistor_THT:R_Axial_DIN0207_L6.3mm_D2.5mm_P10.16mm_Horizontal, F.Cu at (360.7, 119.4)
- added R121: 47k, Resistor_THT:R_Axial_DIN0207_L6.3mm_D2.5mm_P10.16mm_Horizontal, F.Cu at (332.7, 118.1)
- added R122: 150, Resistor_THT:R_Axial_DIN0207_L6.3mm_D2.5mm_P10.16mm_Horizontal, F.Cu at (349.2, 123.2)
- added R123: 1k, Resistor_THT:R_Axial_DIN0207_L6.3mm_D2.5mm_P10.16mm_Horizontal, F.Cu at (349.2, 126.5)
- added R124: 1k, Resistor_THT:R_Axial_DIN0207_L6.3mm_D2.5mm_P10.16mm_Horizontal, F.Cu at (332.7, 131.4)
- added R130: 10R, Resistor_THT:R_Axial_DIN0207_L6.3mm_D2.5mm_P10.16mm_Horizontal, F.Cu at (360.7, 99.1)
- added R131: 270k, Resistor_THT:R_Axial_DIN0207_L6.3mm_D2.5mm_P10.16mm_Horizontal, F.Cu at (339.1, 96.5)
- added R132: 150, Resistor_THT:R_Axial_DIN0207_L6.3mm_D2.5mm_P10.16mm_Horizontal, F.Cu at (339.1, 102.2)
- added R133: 1k, Resistor_THT:R_Axial_DIN0207_L6.3mm_D2.5mm_P10.16mm_Horizontal, F.Cu at (349.2, 108.0)
- added R140: 10R, Resistor_THT:R_Axial_DIN0207_L6.3mm_D2.5mm_P10.16mm_Horizontal, F.Cu at (360.7, 81.3)
- added R141: 270k, Resistor_THT:R_Axial_DIN0207_L6.3mm_D2.5mm_P10.16mm_Horizontal, F.Cu at (339.1, 78.7)
- added R142: 150, Resistor_THT:R_Axial_DIN0207_L6.3mm_D2.5mm_P10.16mm_Horizontal, F.Cu at (339.1, 84.5)
- added R143: 1k, Resistor_THT:R_Axial_DIN0207_L6.3mm_D2.5mm_P10.16mm_Horizontal, F.Cu at (349.2, 90.2)
- added R220: 180, Resistor_THT:R_Axial_DIN0207_L6.3mm_D2.5mm_P10.16mm_Horizontal, F.Cu at (327.7, 118.1)
- added R221: 10k, Resistor_THT:R_Axial_DIN0207_L6.3mm_D2.5mm_P10.16mm_Horizontal, F.Cu at (314.3, 127.6)
- added R222: 1k, Resistor_THT:R_Axial_DIN0207_L6.3mm_D2.5mm_P10.16mm_Horizontal, F.Cu at (314.3, 131.4)
- added R230: 180, Resistor_THT:R_Axial_DIN0207_L6.3mm_D2.5mm_P10.16mm_Horizontal, F.Cu at (327.7, 96.5)
- added R231: 10k, Resistor_THT:R_Axial_DIN0207_L6.3mm_D2.5mm_P10.16mm_Horizontal, F.Cu at (314.3, 104.8)
- added R232: 1k, Resistor_THT:R_Axial_DIN0207_L6.3mm_D2.5mm_P10.16mm_Horizontal, F.Cu at (314.3, 108.0)
- added R240: 180, Resistor_THT:R_Axial_DIN0207_L6.3mm_D2.5mm_P10.16mm_Horizontal, F.Cu at (327.7, 78.7)
- added R241: 10k, Resistor_THT:R_Axial_DIN0207_L6.3mm_D2.5mm_P10.16mm_Horizontal, F.Cu at (314.3, 87.0)
- added R242: 1k, Resistor_THT:R_Axial_DIN0207_L6.3mm_D2.5mm_P10.16mm_Horizontal, F.Cu at (314.3, 90.2)
- added R900: 3k3, Resistor_THT:R_Axial_DIN0207_L6.3mm_D2.5mm_P10.16mm_Horizontal, F.Cu at (373.4, 52.1)
- added R901: 390, Resistor_THT:R_Axial_DIN0207_L6.3mm_D2.5mm_P10.16mm_Horizontal, F.Cu at (373.4, 55.9)
- added R902: 68R, Resistor_THT:R_Axial_DIN0207_L6.3mm_D2.5mm_P10.16mm_Horizontal, F.Cu at (355.6, 73.0)
- added R903: 3k3, Resistor_THT:R_Axial_DIN0207_L6.3mm_D2.5mm_P10.16mm_Horizontal, F.Cu at (323.2, 69.8)
- added U220: 4N35, Package_DIP:DIP-6_W7.62mm_Socket_LongPads, F.Cu at (327.7, 122.6)
- added U230: 4N35, Package_DIP:DIP-6_W7.62mm_Socket_LongPads, F.Cu at (327.7, 99.7)
- added U240: 4N35, Package_DIP:DIP-6_W7.62mm_Socket_LongPads, F.Cu at (327.7, 81.9)
- added U900: LM317, Package_TO_SOT_THT:TO-220-3_Horizontal_TabDown, F.Cu at (375.9, 57.1)
- added U901: L78L05_TO92, Package_TO_SOT_THT:TO-92_Inline_Wide, F.Cu at (351.2, 58.4)
- added U902: HCPL7510, Package_DIP:DIP-8_W7.62mm_Socket_LongPads, F.Cu at (341.0, 66.7)
- U3: footprint Package_DIP:DIP-28_W7.62mm -> Package_DIP:DIP-28_W7.62mm_Socket_LongPads
- moved DS1 299.9 mm to (281.9, 55.9), turned to -90 degrees
- moved F1 296.8 mm to (367.3, 36.8)
- moved J5 293.2 mm to (353.1, 36.8)
- moved J4 283.2 mm to (342.9, 36.8)
- moved J6 273.1 mm to (332.7, 36.8)
- moved SW1 229.7 mm to (259.2, 137.9)
- moved U3 221.1 mm to (295.3, 74.9)
- moved U9 220.6 mm to (290.2, 46.4)
- moved R212 61.2 mm to (314.3, 154.3)
- moved R210 61.0 mm to (327.7, 141.0)
- moved Q110 61.0 mm to (375.9, 142.2)
- moved C110 61.0 mm to (348.6, 152.7)
- moved Q111 61.0 mm to (345.4, 142.2)
- moved Q112 61.0 mm to (353.1, 142.2)
- moved Q113 61.0 mm to (353.1, 152.4)
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Connections:
- net /Out_{1} renamed /H Bridge/Out_{1}
- F1 pad 1: Net-(J5-Pin_1) -> Net-(J5-Pin_2)
- J4 pad 1: /Out_{2} -> /H Bridge/Out_{2}
- J5 pad 1: Net-(J5-Pin_1) -> GNDPWR
- J5 pad 2: GNDPWR -> Net-(J5-Pin_2)
- R212 pad 1: P1B -> /H Bridge/P1B
Routing:
- net (no net): track 245.0 -> 1.15 mm
- net /H Bridge/Out_{1}: track 11.3 -> 189.7 mm
- net /H Bridge/Out_{2}: track 0.00 -> 171.3 mm
- net +12V: track 0.00 -> 159.7 mm
- net +24V: track 0.00 -> 120.5 mm
- net /H Bridge/GNDPWR_{out}: track 0.00 -> 58.3 mm
- net Net-(U902-V_{IN+}): track 0.00 -> 27.4 mm
- net Net-(D901-A): track 0.00 -> 26.7 mm
- net Net-(Q121-C): track 0.00 -> 24.6 mm
- net Net-(Q122-B): track 0.00 -> 22.3 mm
- net Net-(U901-VO): track 0.00 -> 18.0 mm
- net Net-(Q121-B): track 0.00 -> 17.0 mm
- net Net-(D120-K): track 0.00 -> 15.9 mm
- net Net-(Q141-B): track 0.00 -> 14.6 mm
- net Net-(Q131-B): track 0.00 -> 14.6 mm
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Other:
- board size 160 x 100 mm -> 160 x 130 mm

Commit message: Update to v 9.0
Parts:
- moved U9 16.9 mm to (303.4, 35.8)
Routing:
- net SCL: track 0.64 -> 0.00 mm

Commit message: Update 090725
New footprints added
Schematic made into sub schematics
PCB needs work
Component references need to be sorted for the most part
Parts:
- added C2: 100nF, Capacitor_THT:C_Rect_L7.2mm_W2.5mm_P5.00mm_FKS2_FKP2_MKS2_MKP2, F.Cu at (130.3, 50.8)
- added REF**: Heatsink_Fisher_FK237SA220H, User:Heatsink_Fisher_FK237SA220O, F.Cu at (214.6, 108.8)
- added REF**: Heatsink_Fisher_FK237SA220H, User:Heatsink_Fisher_FK237SA220O, F.Cu at (214.6, 129.2)
- added REF**: MountingHole_3.2mm_M3_Pad_TopBottom, MountingHole:MountingHole_3.2mm_M3_Pad_TopBottom, F.Cu at (233.7, 160.0)
- added REF**: Heatsink_Fisher_FK237SA220H, User:Heatsink_Fisher_FK237SA220O, F.Cu at (214.6, 152.0)
- added REF**: MountingHole_3.2mm_M3_Pad_TopBottom, MountingHole:MountingHole_3.2mm_M3_Pad_TopBottom, F.Cu at (233.7, 35.6)
- added REF**: MountingHole_3.2mm_M3_Pad_TopBottom, MountingHole:MountingHole_3.2mm_M3_Pad_TopBottom, F.Cu at (86.4, 35.6)
- added REF**: Heatsink_Fisher_FK237SA220H, User:Heatsink_Fisher_FK237SA220O, F.Cu at (214.6, 91.1)
- added REF**: Heatsink_Fisher_FK237SA220H, User:Heatsink_Fisher_FK237SA220O, F.Cu at (214.6, 66.9)
- DS1: footprint Display:WC1602A -> User:Powertip_PC1602
- SW1: footprint Rotary_Encoder:RotaryEncoder_Alps_EC11E-Switch_Vertical_H20mm -> User:RotaryEncoder_Bourns-Switch_Vertical_H20mm
- moved DS1 207.6 mm to (84.6, 120.3)
- moved U9 175.3 mm to (129.0, 54.0)
- moved U3 165.8 mm to (129.5, 77.5)
- moved C900 165.4 mm to (224.5, 46.0)
- moved F1 165.4 mm to (201.9, 35.5)
- moved J5 165.4 mm to (187.7, 35.5)
- moved J6 165.4 mm to (167.3, 35.5)
- moved J4 165.4 mm to (177.5, 35.5)
- moved C906 165.4 mm to (164.2, 65.0)
- moved C907 165.4 mm to (161.0, 65.0)
- moved C110 165.4 mm to (183.2, 152.7)
- moved C120 165.4 mm to (183.2, 129.8)
- moved C901 165.4 mm to (194.0, 55.9)
- moved C902 165.4 mm to (194.0, 62.2)
- moved D110 165.4 mm to (187.7, 147.3)
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Connections:
- U3 pad 13: P1A -> /H Bridge/P1A
- U3 pad 22: P1C -> /H Bridge/P1D
- U3 pad 23: P1B -> /H Bridge/P1B
- U3 pad 25: P1D -> /H Bridge/P1C
Routing:
- net SDO: track 0.00 -> 82.6 mm
- net /H Bridge/P1B: track 0.00 -> 74.2 mm
- net Net-(DS1-RS): track 0.00 -> 66.8 mm
- net +12V: track 159.7 -> 220.5 mm
- net SDA/SDI: track 0.00 -> 60.2 mm
- net Net-(DS1-E): track 0.00 -> 57.8 mm
- net SCL: track 0.00 -> 56.0 mm
- net Net-(DS1-D4): track 0.00 -> 51.6 mm
- net /H Bridge/P1A: track 0.00 -> 47.4 mm
- net /H Bridge/P1D: track 0.00 -> 47.4 mm
- net DISP: track 0.00 -> 46.8 mm
- net RA4: track 0.00 -> 40.6 mm
- net uRX: track 0.00 -> 39.1 mm
- net uTX: track 0.00 -> 34.4 mm
- net +5V: track 10.9 -> 45.1 mm
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Other:
- board size 160 x 130 mm -> 160 x 135.1 mm

Commit message: Almost done
Schematic done
PCB missing ground planes
Need Coopilot review
Parts:
- removed C1, C10, C13, C2, C5, C7: 100nF, Capacitor_THT:C_Rect_L7.2mm_W2.5mm_P5.00mm_FKS2_FKP2_MKS2_MKP2
- removed C3: 470nF, Capacitor_THT:C_Rect_L7.2mm_W2.5mm_P5.00mm_FKS2_FKP2_MKS2_MKP2
- removed DS1: WC1602A, User:Powertip_PC1602
- removed J2: Conn_01x06_Pin, Connector_PinHeader_2.54mm:PinHeader_1x06_P2.54mm_Vertical
- removed J3: USB_B, Connector_USB:USB_B_TE_5787834_Vertical
- removed R19, R29, R32, R39, R4, R43, R5: 10k, Resistor_THT:R_Axial_DIN0207_L6.3mm_D2.5mm_P10.16mm_Horizontal
- removed R23, R27, R41, R42: 1k, Resistor_THT:R_Axial_DIN0207_L6.3mm_D2.5mm_P10.16mm_Horizontal
- removed the REF** at (233.7, 160.0)
- removed the REF** at (233.7, 35.6)
- removed the REF** at (86.4, 35.6)
- removed the REF** at (214.6, 66.9)
- removed RV1: 50k, Potentiometer_THT:Potentiometer_Piher_PT-10-V05_Vertical
- removed SW1: RotaryEncoder_Switch_MP, User:RotaryEncoder_Bourns-Switch_Vertical_H20mm
- removed U3: PIC18F26K22-xSP, Package_DIP:DIP-28_W7.62mm_Socket_LongPads
- removed U4: MCP2221AxP, Package_DIP:DIP-14_W7.62mm_Socket_LongPads
- removed U9: 74AHC595, Package_DIP:DIP-16_W7.62mm_Socket_LongPads
- added C250: 100nF, Capacitor_THT:C_Rect_L7.2mm_W2.5mm_P5.00mm_FKS2_FKP2_MKS2_MKP2, F.Cu at (155.6, 49.5)
- added C300: 100nF, Capacitor_THT:C_Rect_L7.2mm_W2.5mm_P5.00mm_FKS2_FKP2_MKS2_MKP2, F.Cu at (130.9, 54.6)
- added C310: 100nF, Capacitor_THT:C_Rect_L7.2mm_W2.5mm_P5.00mm_FKS2_FKP2_MKS2_MKP2, F.Cu at (140.3, 118.7)
- added C311: 100nF, Capacitor_THT:C_Rect_L7.2mm_W2.5mm_P5.00mm_FKS2_FKP2_MKS2_MKP2, F.Cu at (140.3, 121.9)
- added C312: 100nF, Capacitor_THT:C_Rect_L7.2mm_W2.5mm_P5.00mm_FKS2_FKP2_MKS2_MKP2, F.Cu at (140.3, 125.1)
- added C400: 100nF, Capacitor_THT:C_Rect_L7.2mm_W2.5mm_P5.00mm_FKS2_FKP2_MKS2_MKP2, F.Cu at (142.2, 101.6)
- added C410: 470nF, Capacitor_THT:C_Rect_L7.2mm_W2.5mm_P5.00mm_FKS2_FKP2_MKS2_MKP2, F.Cu at (126.4, 141.1)
- added C411: 100nF, Capacitor_THT:C_Rect_L7.2mm_W2.5mm_P5.00mm_FKS2_FKP2_MKS2_MKP2, F.Cu at (141.0, 141.0)
- added DS300: WC1602A, User:Powertip_PC1602, F.Cu at (83.7, 124.1)
- added J400: Conn_01x05_Pin, Connector_PinSocket_2.54mm:PinSocket_1x05_P2.54mm_Horizontal, F.Cu at (161.3, 40.6)
- added J410: Conn_01x06_Pin, Connector_PinSocket_2.54mm:PinSocket_1x06_P2.54mm_Vertical, F.Cu at (133.3, 143.5)
- added J411: USB_B, Connector_USB:USB_B_TE_5787834_Vertical, F.Cu at (134.0, 154.9)
- added R250: 1k, Resistor_THT:R_Axial_DIN0207_L6.3mm_D2.5mm_P10.16mm_Horizontal, F.Cu at (168.9, 49.5)
- added R251: 10k, Resistor_THT:R_Axial_DIN0207_L6.3mm_D2.5mm_P10.16mm_Horizontal, F.Cu at (158.8, 44.5)
- added R300: 50k, Potentiometer_THT:Potentiometer_Bourns_3339P_Vertical_HandSoldering, F.Cu at (127.0, 48.9)
- added R310: 10k, Resistor_THT:R_Axial_DIN0207_L6.3mm_D2.5mm_P10.16mm_Horizontal, F.Cu at (113.7, 135.9)
- added R311: 10k, Resistor_THT:R_Axial_DIN0207_L6.3mm_D2.5mm_P10.16mm_Horizontal, F.Cu at (117.5, 135.9)
- added R312: 10k, Resistor_THT:R_Axial_DIN0207_L6.3mm_D2.5mm_P10.16mm_Horizontal, F.Cu at (121.3, 135.9)
- added R313: 1k, Resistor_THT:R_Axial_DIN0207_L6.3mm_D2.5mm_P10.16mm_Horizontal, F.Cu at (137.8, 118.7)
- added R314: 1k, Resistor_THT:R_Axial_DIN0207_L6.3mm_D2.5mm_P10.16mm_Horizontal, F.Cu at (127.6, 121.9)
- added R315: 1k, Resistor_THT:R_Axial_DIN0207_L6.3mm_D2.5mm_P10.16mm_Horizontal, F.Cu at (127.6, 125.1)
- added R400: 10k, Resistor_THT:R_Axial_DIN0207_L6.3mm_D2.5mm_P10.16mm_Horizontal, F.Cu at (123.8, 96.5)
- added R401: 10k, Resistor_THT:R_Axial_DIN0207_L6.3mm_D2.5mm_P10.16mm_Horizontal, F.Cu at (123.8, 109.2)
- added R410: 10k, Resistor_THT:R_Axial_DIN0207_L6.3mm_D2.5mm_P10.16mm_Horizontal, F.Cu at (141.0, 128.3)
- added SW310: RotaryEncoder_Switch_MP, User:RotaryEncoder_Bourns-Switch_Vertical_H20mm, F.Cu at (94.6, 137.2)
- added U300: 74AHC595, Package_DIP:DIP-16_W7.62mm_Socket_LongPads, F.Cu at (129.5, 57.8)
- added U400: PIC18F26K22-xSP, Package_DIP:DIP-28_W7.62mm_Socket_LongPads, F.Cu at (129.5, 81.3)
- added U410: MCP2221AxP, Package_DIP:DIP-14_W7.62mm_Socket_LongPads, F.Cu at (137.2, 146.1)
- J1: value Conn_01x05_Pin -> Conn_01x02_Socket; footprint Connector_PinSocket_2.54mm:PinSocket_1x05_P2.54mm_Horizontal -> Connector_Phoenix_MC_HighVoltage:PhoenixContact_MCV_1,5_2-G-5.08_1x02_P5.08mm_Vertical
- moved J1 103.6 mm to (139.7, 35.6)
- moved D900 0.70 mm to (205.7, 62.9)
- moved C907 0.34 mm to (160.7, 65.0)
- moved D110 0.29 mm to (188.0, 147.3)
- moved D120 0.29 mm to (188.0, 124.5)
- moved D901 0.29 mm to (205.7, 59.1)
- moved J4 0.29 mm to (177.8, 35.5)
- moved J5 0.29 mm to (188.0, 35.5)
- moved Q112 0.29 mm to (188.0, 142.2)
- moved Q113 0.29 mm to (188.0, 152.4)
- moved Q122 0.29 mm to (188.0, 119.4)
- moved Q123 0.29 mm to (188.0, 129.5)
- moved Q131 0.29 mm to (188.0, 99.1)
- moved Q132 0.29 mm to (188.0, 107.3)
- moved Q141 0.29 mm to (188.0, 81.3)
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Connections:
- net /PSU/AN0 renamed /MCU & USB/AN0
- J1 pad 1: V_{PP} -> +5V
- J1 pad 2: +5V -> GNDD
Routing:
- net +5V: track 45.1 -> 311.1 mm
- net PGC: track 0.00 -> 83.0 mm
- net SDO: track 82.6 -> 0.00 mm
- net /Disp & encoder/SDO: track 0.00 -> 82.6 mm
- net T1CLK: track 0.00 -> 77.1 mm, vias 0 -> 2
- net PGD: track 0.00 -> 73.1 mm
- net Net-(DS1-RS): track 66.8 -> 0.00 mm
- net Net-(DS300-RS): track 0.00 -> 66.8 mm
- net /Disp & encoder/SDA/SDI: track 0.00 -> 61.0 mm
- net SDA/SDI: track 60.2 -> 0.00 mm
- net V_{PP}: track 0.00 -> 57.9 mm
- net Net-(DS300-E): track 0.00 -> 57.8 mm
- net Net-(DS1-E): track 57.8 -> 0.00 mm
- net /Disp & encoder/SCL: track 0.00 -> 57.2 mm
- net SCL: track 56.0 -> 0.00 mm
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
Commit message: Few changes made
Parts:
- added L1: L_Ferrite_Small, Resistor_THT:R_Axial_DIN0411_L9.9mm_D3.6mm_P12.70mm_Horizontal, F.Cu at (142.9, 161.9)
- renumbered U110 to U210

Commit message: V 1.0 fabrication output
V 1.0 ready for fabrication
Parts:
- removed L1: L_Ferrite_Small, Resistor_THT:R_Axial_DIN0411_L9.9mm_D3.6mm_P12.70mm_Horizontal
- added G***: LOGO, User:logo, B.Cu at (84.1, 90.2)
- added L410: L_Ferrite_Small, Resistor_THT:R_Axial_DIN0411_L9.9mm_D3.6mm_P12.70mm_Horizontal, F.Cu at (126.6, 150.5)
- added REF**: Heatsink_Fisher_FK237SA220H, User:Heatsink_Fisher_FK237SA220O, F.Cu at (198.7, 55.5)
- added REF**: MountingHole_3.2mm_M3_ISO7380_Pad_TopOnly, MountingHole:MountingHole_3.2mm_M3_ISO7380_Pad_TopOnly, F.Cu at (72.0, 145.9)
- added REF**: MountingHole_3.2mm_M3_ISO7380_Pad_TopOnly, MountingHole:MountingHole_3.2mm_M3_ISO7380_Pad_TopOnly, F.Cu at (217.0, 145.9)
- added REF**: MountingHole_3.2mm_M3_ISO7380_Pad_TopOnly, MountingHole:MountingHole_3.2mm_M3_ISO7380_Pad_TopOnly, F.Cu at (72.0, 25.9)
- added REF**: MountingHole_3.2mm_M3_ISO7380_Pad_TopOnly, MountingHole:MountingHole_3.2mm_M3_ISO7380_Pad_TopOnly, F.Cu at (217.0, 25.9)
- Q110, Q120, Q130, Q140, U900: footprint Package_TO_SOT_THT:TO-220-3_Horizontal_TabDown -> User:TO-220-3_Horizontal_TabDown_HoleToCenter
- moved REF** 19.9 mm to (198.7, 79.6)
- moved D110 19.9 mm to (171.7, 135.9)
- moved Q112 19.9 mm to (171.7, 130.8)
- moved Q113 19.9 mm to (171.7, 141.0)
- moved Q131 19.9 mm to (171.7, 87.6)
- moved Q141 19.9 mm to (171.7, 69.8)
- moved R110 19.9 mm to (179.3, 130.8)
- moved R112 19.9 mm to (167.9, 134.6)
- moved R113 19.9 mm to (167.9, 137.9)
- moved R123 19.9 mm to (167.9, 115.1)
- moved R130 19.9 mm to (179.3, 87.6)
- moved R133 19.9 mm to (167.9, 96.5)
- moved R140 19.9 mm to (179.3, 69.8)
- moved R143 19.9 mm to (167.9, 78.7)
- moved C904 19.9 mm to (167.9, 55.2)
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Routing:
- net +5V: track 311.1 -> 331.4 mm
- net GNDD: track 8.01 -> 26.6 mm
- net Net-(DS300-E): track 57.8 -> 44.1 mm
- net Net-(R312-Pad1): track 35.9 -> 49.3 mm
- net Net-(DS300-D4): track 51.6 -> 40.8 mm
- net RA4: track 40.6 -> 48.5 mm
- net Net-(DS300-RS): track 66.8 -> 61.5 mm
- net /H Bridge/Out_{1}: track 191.0 -> 194.6 mm, vias 0 -> 12
- net Net-(DS300-VO): track 18.5 -> 16.6 mm
- net Net-(DS300-D7): track 29.9 -> 28.3 mm
- net +24V: track 143.7 -> 142.3 mm, vias 0 -> 24
- net Net-(DS300-D5): track 30.8 -> 31.3 mm
- net +12V: vias 0 -> 12
- net /H Bridge/Out_{2}: vias 0 -> 12
- added copper zone on B.Cu, net +12V
- added copper zone on F.Cu, net +12V
- added copper zone on B.Cu, net +24V
- added copper zone on F.Cu, net +24V
- added copper zone on B.Cu, net /H Bridge/Out_{1}
- added copper zone on F.Cu, net /H Bridge/Out_{1}
- added copper zone on B.Cu, net /H Bridge/Out_{2}
- added copper zone on F.Cu, net /H Bridge/Out_{2}
- added copper zone on F.Cu, net GNDD
- added copper zone on F.Cu, net GNDPWR
- added copper zone on F.Cu, net Net-(J411-Shield)
Other:
- board size 160 x 135.1 mm -> 160 x 135.3 mm
- board text added: "Motor Control v 1.0"
