File: Motor Control.kicad_pcb (KiCad board)
At the start: 2 copper layers, 160 x 135.3 mm, 118 parts, among them J1 Conn_01x02_Socket, J4 Conn_01x02_Socket, J400 Conn_01x05_Pin, J410 Conn_01x06_Pin, J411 USB_B, J5 Conn_01x02_Socket, J6 Conn_01x02_Socket, Q110 IRLZ44N, Q111 BC557, Q112 BC547, Q113 BC557, Q120 IRLZ44N, Q121 BC557, Q122 BC547, Q123 BC557, Q130 IRLZ44N, Q131 BC547, Q132 BC557, Q140 IRLZ44N, Q141 BC547, Q142 BC557, Q210 BC547, Q220 BC547, Q230 BC547, Q240 BC547, SW310 RotaryEncoder_Switch_MP, U210 4N35, U220 4N35, U230 4N35, U240 4N35, U300 74AHC595, U400 PIC18F26K22-xSP, U410 MCP2221AxP, U900 LM317, U901 L78L05_TO92, U902 HCPL7510

Commit message: V 2.0
Parts:
- added C401: 100nF, Capacitor_THT:C_Rect_L7.2mm_W2.5mm_P5.00mm_FKS2_FKP2_MKS2_MKP2, F.Cu at (123.8, 71.8)
- added J401: Conn_01x04_Socket, Connector_PinSocket_2.54mm:PinSocket_1x04_P2.54mm_Horizontal, F.Cu at (74.9, 123.2)
- added R300: 10k, Resistor_THT:R_Axial_DIN0207_L6.3mm_D2.5mm_P10.16mm_Horizontal, F.Cu at (123.8, 61.0)
- added R402: 10k, Resistor_THT:R_Axial_DIN0207_L6.3mm_D2.5mm_P10.16mm_Horizontal, F.Cu at (127.0, 68.6)
- added R403: 100R, Resistor_THT:R_Axial_DIN0207_L6.3mm_D2.5mm_P10.16mm_Horizontal, F.Cu at (110.5, 71.8)
- C110, C120: value 1uF -> 2.2uF
- C900: value 330uF -> 220uF
- C901, C902: value 1uF -> 10uF
- R301: renamed from R300; value 50k -> 20k
- U400: value PIC18F26K22-xSP -> PIC18F27Q43-xSP
- U901: value L78L05_TO92 -> L78L05
- moved SW310 23.1 mm to (102.1, 130.1), turned to 180 degrees
- moved R410 15.3 mm to (111.1, 121.3), turned to 0 degrees
- moved R310 13.1 mm to (95.2, 137.2)
- moved R311 13.1 mm to (99.1, 137.2)
- moved R312 13.1 mm to (102.9, 137.2)
- moved R231 8.35 mm to (132.7, 101.6)
- moved R401 8.14 mm to (105.7, 90.2)
- moved C410 5.43 mm to (109.2, 134.7)
- moved REF** 5.38 mm to (198.4, 145.6)
- moved REF** 5.38 mm to (198.4, 122.7)
- moved REF** 5.34 mm to (198.4, 102.4)
- moved C120 5.24 mm to (167.0, 123.5)
- moved C411 5.24 mm to (124.5, 134.6)
- moved D110 5.24 mm to (171.4, 141.0)
- moved Q113 5.24 mm to (171.4, 146.1)
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Connections:
- net Net-(J411-D+) renamed /MCU & USB/D+
- net Net-(J411-D-) renamed /MCU & USB/D-
- net Net-(U400-RA2) renamed /MCU & USB/V_{REF-}
- C907 pad 1: /MCU & USB/AN0 -> /MCU & USB/AN
- DS300 pad 11: Net-(DS300-D4) -> /Disp & encoder/D4_{disp}
- DS300 pad 12: Net-(DS300-D5) -> /Disp & encoder/D5_{disp}
- DS300 pad 13: Net-(DS300-D6) -> /Disp & encoder/D6_{disp}
- DS300 pad 14: Net-(DS300-D7) -> /Disp & encoder/D7_{disp}
- DS300 pad 4: Net-(DS300-RS) -> /Disp & encoder/RS_{disp}
- DS300 pad 6: Net-(DS300-E) -> /Disp & encoder/E_{disp}
- J400 pad 4: PGD -> MOSI_{1}/PGD
- J400 pad 5: PGC -> SCL_{1}/PGC
- R410 pad 1: RA4 -> RA6
- R903 pad 1: /MCU & USB/AN0 -> /MCU & USB/AN
- U300 pad 1: Net-(DS300-D5) -> unconnected-(U300-QB-Pad1)
- U300 pad 10: GNDD -> Net-(U300-~{SRCLR})
- U300 pad 11: /Disp & encoder/SCL -> SCL_{1}/PGC
- U300 pad 12: /Disp & encoder/DISP -> /Disp & encoder/DISP_{SS}
- U300 pad 14: /Disp & encoder/SDO -> MOSI_{1}/PGD
- U300 pad 15: Net-(DS300-D4) -> unconnected-(U300-QA-Pad15)
- U300 pad 2: Net-(DS300-D6) -> /Disp & encoder/RS_{disp}
- U300 pad 3: Net-(DS300-D7) -> /Disp & encoder/E_{disp}
- U300 pad 4: unconnected-(U300-QE-Pad4) -> /Disp & encoder/D4_{disp}
- U300 pad 5: Net-(DS300-RS) -> /Disp & encoder/D5_{disp}
- U300 pad 6: unconnected-(U300-QG-Pad6) -> /Disp & encoder/D6_{disp}
- U300 pad 7: Net-(DS300-E) -> /Disp & encoder/D7_{disp}
- U300 pad 9: /Disp & encoder/SDA/SDI -> unconnected-(U300-QH&apos;-Pad9)
- U400 pad 1: V_{PP} -> Net-(U400-~{MCLR}/VPP/RE3)
- U400 pad 10: unconnected-(U400-RA6/OSC2_CLKOUT-Pad10) -> RA6
- U400 pad 11: T1CLK -> Net-(J401-Pin_1)
- U400 pad 12: /Disp & encoder/DISP -> Net-(J401-Pin_2)
- U400 pad 13: /H Bridge/P1A -> Net-(J401-Pin_3)
- U400 pad 14: /Disp & encoder/SCL -> Net-(J401-Pin_4)
- U400 pad 15: /Disp & encoder/SDA/SDI -> uTX
- U400 pad 16: /Disp & encoder/SDO -> uRX
- U400 pad 17: uTX -> /H Bridge/P1B
- U400 pad 18: uRX -> /H Bridge/P1D
- U400 pad 2: /MCU & USB/AN0 -> T1CLK
- U400 pad 21: /Disp & encoder/SWS -> unconnected-(U400-RB0-Pad21)
- U400 pad 22: /H Bridge/P1D -> /H Bridge/P1A
- U400 pad 23: /H Bridge/P1B -> /H Bridge/P1C
- U400 pad 24: /Disp & encoder/SWA -> GNDD
- U400 pad 25: /H Bridge/P1C -> /MCU & USB/AN
- U400 pad 26: /Disp & encoder/SWB -> /Disp & encoder/DISP_{SS}
- U400 pad 27: PGC -> SCL_{1}/PGC
- U400 pad 28: PGD -> MOSI_{1}/PGD
- U400 pad 6: RA4 -> /Disp & encoder/SWS
- U400 pad 7: ~{SS} -> /Disp & encoder/SWA
- U400 pad 9: unconnected-(U400-RA7/OSC1_CLKIN-Pad9) -> /Disp & encoder/SWB
- U410 pad 8: RA4 -> RA6
Routing:
- net PGC: track 83.0 -> 0.00 mm
- net /Disp & encoder/SDO: track 82.6 -> 0.00 mm
- net MOSI_{1}/PGD: track 0.00 -> 74.6 mm, vias 0 -> 1
- net PGD: track 73.1 -> 0.00 mm
- net SCL_{1}/PGC: track 0.00 -> 66.9 mm
- net Net-(DS300-RS): track 61.5 -> 0.00 mm
- net /Disp & encoder/SDA/SDI: track 61.0 -> 0.00 mm
- net /Disp & encoder/SCL: track 57.2 -> 0.00 mm
- net /Disp & encoder/DISP: track 50.3 -> 0.00 mm
- net Net-(J401-Pin_3): track 0.00 -> 49.3 mm
- net Net-(J401-Pin_4): track 0.00 -> 48.7 mm
- net Net-(J401-Pin_2): track 0.00 -> 48.7 mm
- net RA4: track 48.5 -> 0.00 mm
- net Net-(J401-Pin_1): track 0.00 -> 47.9 mm
- net Net-(DS300-E): track 44.1 -> 0.00 mm
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- added copper zone on B.Cu, net GNDD
- added copper zone on B.Cu, net GNDPWR
- added copper zone on B.Cu, net Net-(J411-Shield)
