File: MCU_USB.kicad_sch (KiCad schematic)
At the start: 15 parts, among them J1 Conn_01x05_Pin, J2 Conn_01x06_Pin, J3 USB_B, J6 Conn_01x02_Socket, U3 PIC18F26K22-xSP, U4 MCP2221AxP

Commit message: Almost done
Schematic done
PCB missing ground planes
Need Coopilot review
Parts:
- added C411: 100nF, Capacitor_THT:C_Rect_L7.2mm_W2.5mm_P5.00mm_FKS2_FKP2_MKS2_MKP2, symbol Device:C_Small
- added J1: Conn_01x02_Socket, Connector_Phoenix_MC_HighVoltage:PhoenixContact_MCV_1,5_2-G-5.08_1x02_P5.08mm_Vertical, symbol Connector:Conn_01x02_Socket
- J410: renamed from J2; footprint Connector_PinHeader_2.54mm:PinHeader_1x06_P2.54mm_Vertical -> Connector_PinSocket_2.54mm:PinSocket_1x06_P2.54mm_Vertical
- renumbered C13 to C250, C1 to C400, C3 to C410, J1 to J400, J3 to J411, R42 to R250, R43 to R251, R4 to R400, R5 to R401, R19 to R410, U3 to U400, U4 to U410
Connections:
- net +5V: now also C411.1, J1.1 (Pin_1); no longer C410.1
- net GNDD: now also C410.2, J411.4 (GND), L1.2, U410.14 (VSS), C411.2, J1.2 (Pin_2)
- net at U410.11 (VUSB): now also C410.1; no longer C410.2
- no-connect marks 8 -> 12
Other:
- moved on the sheet: C410, J410, R410

Commit message: V 1.0 fabrication output
V 1.0 ready for fabrication
Parts:
- L410: renamed from L1; footprint (none) -> Resistor_THT:R_Axial_DIN0411_L9.9mm_D3.6mm_P12.70mm_Horizontal
Other:
- company: (none) -> AARHUS TECH
- title: (none) -> Motor Control
Changed lines of the file:
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@@
 	(generator_version "9.0")
 	(paper "A4")
+	(title_block
+		(title "Motor Control")
+		(rev "1.0")
+		(company "AARHUS TECH")
+	)
 	(junction
 		(at 69.85 109.22)
@@
 		(on_board yes)
 		(dnp no)
-		(property "Reference" "L1"
+		(property "Reference" "L410"
 			(at 170.18 88.8999 0)
 			(effects
@@
 			)
 		)
-		(property "Footprint" ""
+		(property "Footprint" "Resistor_THT:R_Axial_DIN0411_L9.9mm_D3.6mm_P12.70mm_Horizontal"
 			(at 171.45 90.17 0)
 			(effects
@@
 			(project "Motor Control"
 				(path "/287fa568-d091-4161-b3b2-3036dfbfe9fa/47a78832-f428-42bb-9cda-183aace586bf"
-					(reference "L1")
+					(reference "L410")
 					(unit 1)
 				)

Commit message: Partnumbers
Parts:
- U400: Part number (none) -> 887-7252; Supplier (none) -> RS
- U410: Part number (none) -> 171-7757; Supplier (none) -> RS

Commit message: BOM
Parts:
- C250, C400, C411: Part number (none) -> 135-8304; Supplier (none) -> RS
- C410: Part number (none) -> 172-5820; Supplier (none) -> RS
- J400: Part number (none) -> 233-9362; Supplier (none) -> RS
- J411: Part number (none) -> 1076666; Supplier (none) -> Farnell
- L410: Part number (none) -> 467-3315; Supplier (none) -> RS
- R250: Part number (none) -> 05.000.0410; Supplier (none) -> Cypax
- R251, R400, R401, R410: Part number (none) -> 05.000.0510; Supplier (none) -> Cypax
Changed lines of the file:
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@@
 			)
 		)
-		(property "Part number" ""
+		(property "Part number" "172-5820"
 			(at 204.47 57.15 90)
 			(effects
@@
 			)
 		)
-		(property "Supplier" ""
+		(property "Supplier" "RS"
 			(at 204.47 57.15 90)
 			(effects
@@
 			)
 		)
-		(property "Part number" ""
+		(property "Part number" "05.000.0510 "
 			(at 204.47 128.27 0)
 			(effects
@@
 			)
 		)
-		(property "Supplier" ""
+		(property "Supplier" "Cypax"
 			(at 204.47 128.27 0)
 			(effects
@@
 			)
 		)
-		(property "Part number" ""
+		(property "Part number" "135-8304"
 			(at 191.77 128.27 0)
 			(effects
@@
 			)
 		)
-		(property "Supplier" ""
+		(property "Supplier" "RS"
 			(at 191.77 128.27 0)
 			(effects
@@
 			)
 		)
-		(property "Part number" ""
+		(property "Part number" "05.000.0510 "
 			(at 69.85 102.87 0)
 			(effects
@@
 			)
 		)
-		(property "Supplier" ""
+		(property "Supplier" "Cypax"
 			(at 69.85 102.87 0)
 			(effects
@@
 			)
 		)
-		(property "Part number" ""
+		(property "Part number" "135-8304"
 			(at 90.17 69.85 0)
 			(effects
@@
 			)
 		)
-		(property "Supplier" ""
+		(property "Supplier" "RS"
 			(at 90.17 69.85 0)
 			(effects
@@
 			)
 		)
-		(property "Part number" ""
+		(property "Part number" "1076666"
 			(at 173.99 74.93 0)
 			(effects
@@
 			)
 		)
-		(property "Supplier" ""
+		(property "Supplier" "Farnell"
 			(at 173.99 74.93 0)
 			(effects
@@
 			)
 		)
-		(property "Part number" ""
+		(property "Part number" "05.000.0410 "
 			(at 196.85 119.38 90)
 			(effects
@@
 			)
 		)
-		(property "Supplier" ""
+		(property "Supplier" "Cypax"
 			(at 196.85 119.38 90)
 			(effects
@@
 			)
 		)
-		(property "Part number" ""
+		(property "Part number" "05.000.0510 "
 			(at 69.85 115.57 0)
 			(effects
@@
 			)
 		)
-		(property "Supplier" ""
+		(property "Supplier" "Cypax"
 			(at 69.85 115.57 0)
 			(effects
@@
 			)
 		)
-		(property "Part number" ""
+		(property "Part number" "135-8304"
 			(at 213.36 52.07 0)
 			(effects
@@
 			)
 		)
-		(property "Supplier" ""
+		(property "Supplier" "RS"
 			(at 213.36 52.07 0)
 			(effects
@@
 			)
 		)
-		(property "Part number" ""
+		(property "Part number" "467-3315"
 			(at 171.45 90.17 0)
 			(effects
@@
 			)
 		)
-		(property "Supplier" ""
+		(property "Supplier" "RS"
 			(at 171.45 90.17 0)
 			(effects
@@
 			)
 		)
-		(property "Part number" ""
+		(property "Part number" "233-9362"
 			(at 95.25 158.75 0)
 			(effects
@@
 			)
 		)
-		(property "Supplier" ""
+		(property "Supplier" "RS"
 			(at 95.25 158.75 0)
 			(effects
@@
 			)
 		)
-		(property "Part number" ""
+		(property "Part number" "05.000.0510 "
 			(at 224.79 71.12 0)
 			(effects
@@
 			)
 		)
-		(property "Supplier" ""
+		(property "Supplier" "Cypax"
 			(at 224.79 71.12 0)
 			(effects

Commit message: V 2.0
Parts:
- added C401: 100nF, Capacitor_THT:C_Rect_L7.2mm_W2.5mm_P5.00mm_FKS2_FKP2_MKS2_MKP2, symbol Device:C
- added J401: Conn_01x04_Socket, Connector_PinSocket_2.54mm:PinSocket_1x04_P2.54mm_Horizontal, symbol Connector:Conn_01x04_Socket
- added R402: 10k, Resistor_THT:R_Axial_DIN0207_L6.3mm_D2.5mm_P10.16mm_Horizontal, symbol Device:R
- added R403: 100R, Resistor_THT:R_Axial_DIN0207_L6.3mm_D2.5mm_P10.16mm_Horizontal, symbol Device:R
- U400: value PIC18F26K22-xSP -> PIC18F27Q43-xSP; Part number 887-7252 -> (none); Supplier RS -> (none)
Connections:
- net AN0 is gone; now on net T1CLK: U400.2 (RA0)
- net SDA/SDI is gone; now on net uTX: U400.15 (RC4)
- net SDO is gone; now on net uRX: U400.16 (RC5)
- net ~{SS} is gone; now on net SWA: U400.7 (RA5)
- net +5V: now also R402.2
- net GNDD: now also U400.24 (RB3), C401.2
- net P1A: now also U400.22 (RB1); no longer U400.13 (RC2)
- net P1B: now also U400.17 (RC6); no longer U400.23 (RB2)
- net P1C: now also U400.23 (RB2); no longer U400.25 (RB4)
- net P1D: now also U400.18 (RC7); no longer U400.22 (RB1)
- net SWA: no longer U400.24 (RB3)
- net SWB: now also U400.9 (RA7/OSC1_CLKIN); no longer U400.26 (RB5)
- net SWS: now also U400.6 (RA4); no longer U400.21 (RB0)
- net T1CLK: no longer U400.11 (RC0/SOSCO)
- net V_{PP}: now also C401.1, R402.1, R403.2; no longer U400.1 (~{MCLR}/VPP/RE3)
- net uRX: no longer U400.18 (RC7)
- net uTX: no longer U400.17 (RC6)
- net D-: now reaches J411.2 (D-), U410.12 (D-)
- net D+: now reaches J411.3 (D+), U410.13 (D+)
- net V_{REF-}: now reaches R400.1, R401.2, U400.4 (RA2)
- net RA6: now reaches U400.10 (RA6/OSC2_CLKOUT)
- net RA6: now also R410.1, U410.8 (GP3)
- net DISP: no longer names the net of U400.12 (RC1/SOSCI)
- net DISP: now also J401.2 (Pin_2)
- net PGC renamed SCL_{1}/PGC
- net PGD renamed MOSI_{1}/PGD
- removed net RA4: R410.1, U400.6 (RA4), U410.8 (GP3)
- net SCL: no longer names the net of U400.14 (RC3)
- net SCL: now also J401.4 (Pin_4)
- new net: R403.1, U400.1 (~{MCLR}/VPP/RE3)
- new net: J401.1 (Pin_1), U400.11 (RC0/SOSCO)
- new net: J401.3 (Pin_3), U400.13 (RC2)
- new net AN: U400.25 (RB4)
- new net DISP_{SS}: U400.26 (RB5)
- no-connect marks 12 -> 11
Other:
- moved on the sheet: R400, R401
