File: PSU.kicad_sch (KiCad schematic)
At the start: 19 parts, among them J5 Conn_01x02_Socket, U900 LM317, U901 L78L05_TO92, U902 HCPL7510

Commit message: Update 090725
New footprints added
Schematic made into sub schematics
PCB needs work
Component references need to be sorted for the most part
Changed lines of the file:
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@@
 (kicad_sch
-	(version 20231120)
+	(version 20250114)
 	(generator "eeschema")
-	(generator_version "8.0")
+	(generator_version "9.0")
 	(paper "A4")
 	(title_block
@@
 		(shape passive)
 		(at 185.42 99.06 180)
-		(fields_autoplaced yes)
 		(effects
 			(font
@@
 		(shape output)
 		(at 252.73 99.06 0)
-		(fields_autoplaced yes)
 		(effects
 			(font

Commit message: V 1.0 fabrication output
V 1.0 ready for fabrication
Parts:
- U900: footprint Package_TO_SOT_THT:TO-220-3_Horizontal_TabDown -> User:TO-220-3_Horizontal_TabDown_HoleToCenter
Changed lines of the file:
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@@
 		(title "Motor Control")
 		(date "2025-07-03")
-		(rev "0.1.0")
+		(rev "1.0")
 		(company "AARHUS TECH")
 	)
@@
 			)
 		)
-		(property "Footprint" "Package_TO_SOT_THT:TO-220-3_Horizontal_TabDown"
+		(property "Footprint" "User:TO-220-3_Horizontal_TabDown_HoleToCenter"
 			(at 93.98 76.2 0)
 			(effects

Commit message: Partnumbers
Parts:
- U900: Part number (none) -> 168-8786; Supplier (none) -> RS
- U901: value L78L05_TO92 -> L78L05; Part number (none) -> 885-5423; Supplier (none) -> RS
- U902: Part number (none) -> 1085055; Supplier (none) -> Farnell

Commit message: BOM
Parts:
- C900: value 330uF -> 220uF; Part number (none) -> 3254121; Supplier (none) -> Farnell
- C901, C902: value 1uF -> 10uF; Part number (none) -> 2901339; Supplier (none) -> Farnell
- C903, C904, C906, C907: Part number (none) -> 135-8304; Supplier (none) -> RS
- C905: Part number (none) -> 134-5708; Supplier (none) -> RS
- D900, D901: Part number (none) -> 00.001.4148; Supplier (none) -> Cypax
- R900, R903: Part number (none) -> 05.000.0433; Supplier (none) -> Cypax
- R901: Part number (none) -> 05.000.0339; Supplier (none) -> Cypax
- R902: Part number (none) -> 05.000.0268; Supplier (none) -> Cypax
Changed lines of the file:
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@@
 			)
 		)
-		(property "Part number" ""
+		(property "Part number" "135-8304"
 			(at 228.6 109.22 0)
 			(effects
@@
 			)
 		)
-		(property "Supplier" ""
+		(property "Supplier" "RS"
 			(at 228.6 109.22 0)
 			(effects
@@
 			)
 		)
-		(property "Value" "1uF"
+		(property "Value" "10uF"
 			(at 134.62 100.7109 0)
 			(effects
@@
 			)
 		)
-		(property "Part number" ""
+		(property "Part number" "2901339"
 			(at 130.81 100.33 0)
 			(effects
@@
 			)
 		)
-		(property "Supplier" ""
+		(property "Supplier" "Farnell"
 			(at 130.81 100.33 0)
 			(effects
@@
 			)
 		)
-		(property "Part number" ""
+		(property "Part number" "00.001.4148"
 			(at 118.11 91.44 90)
 			(effects
@@
 			)
 		)
-		(property "Supplier" ""
+		(property "Supplier" "Cypax"
 			(at 118.11 91.44 90)
 			(effects
@@
 			)
 		)
-		(property "Value" "1uF"
+		(property "Value" "10uF"
 			(at 121.92 109.6009 0)
 			(effects
@@
 			)
 		)
-		(property "Part number" ""
+		(property "Part number" "2901339"
 			(at 118.11 109.22 0)
 			(effects
@@
 			)
 		)
-		(property "Supplier" ""
+		(property "Supplier" "Farnell"
 			(at 118.11 109.22 0)
 			(effects
@@
 			)
 		)
-		(property "Part number" ""
+		(property "Part number" "05.000.0433"
 			(at 241.3 99.06 90)
 			(effects
@@
 			)
 		)
-		(property "Supplier" ""
+		(property "Supplier" "Cypax"
 			(at 241.3 99.06 90)
 			(effects
@@
 			)
 		)
-		(property "Part number" ""
+		(property "Part number" "05.000.0433"
 			(at 93.98 109.22 0)
 			(effects
@@
 			)
 		)
-		(property "Supplier" ""
+		(property "Supplier" "Cypax"
 			(at 93.98 109.22 0)
 			(effects
@@
 			)
 		)
-		(property "Part number" ""
+		(property "Part number" "134-5708"
 			(at 195.58 107.95 0)
 			(effects
@@
 			)
 		)
-		(property "Supplier" ""
+		(property "Supplier" "RS"
 			(at 195.58 107.95 0)
 			(effects
@@
 			)
 		)
-		(property "Part number" ""
+		(property "Part number" "135-8304"
 			(at 250.19 109.22 0)
 			(effects
@@
 			)
 		)
-		(property "Supplier" ""
+		(property "Supplier" "RS"
 			(at 250.19 109.22 0)
 			(effects
@@
 			)
 		)
-		(property "Part number" ""
+		(property "Part number" "00.001.4148"
 			(at 93.98 72.39 0)
 			(effects
@@
 			)
 		)
-		(property "Supplier" ""
+		(property "Supplier" "Cypax"
 			(at 93.98 72.39 0)
 			(effects
@@
 			)
 		)
-		(property "Part number" ""
+		(property "Part number" "05.000.0268 "
 			(at 190.5 99.06 90)
 			(effects
@@
 			)
 		)
-		(property "Supplier" ""
+		(property "Supplier" "Cypax"
 			(at 190.5 99.06 90)
 			(effects
@@
 			)
 		)
-		(property "Part number" ""
+		(property "Part number" "135-8304"
 			(at 143.51 100.33 0)
 			(effects
@@
 			)
 		)
-		(property "Supplier" ""
+		(property "Supplier" "RS"
 			(at 143.51 100.33 0)
 			(effects
@@
 			)
 		)
-		(property "Part number" ""
+		(property "Part number" " 05.000.0339"
 			(at 106.68 91.44 0)
 			(effects
@@
 			)
 		)
-		(property "Supplier" ""
+		(property "Supplier" "Cypax"
 			(at 106.68 91.44 0)
 			(effects
@@
 			)
 		)
-		(property "Value" "330uF"
+		(property "Value" "220uF"
 			(at 77.47 94.3609 0)
 			(effects
@@
 			)
 		)
-		(property "Part number" ""
+		(property "Part number" "3254121"
 			(at 73.66 93.98 0)
 			(effects
@@
 			)
 		)
-		(property "Supplier" ""
+		(property "Supplier" "Farnell"
 			(at 73.66 93.98 0)
 			(effects
@@
 			)
 		)
-		(property "Part number" ""
+		(property "Part number" "135-8304"
 			(at 167.64 100.33 0)
 			(effects
@@
 			)
 		)
-		(property "Supplier" ""
+		(property "Supplier" "RS"
 			(at 167.64 100.33 0)
 			(effects

Commit message: V 2.0
Connections:
- net AN0 renamed AN
Changed lines of the file:
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@@
 		)
 	)
-	(hierarchical_label "AN0"
+	(hierarchical_label "AN"
 		(shape output)
 		(at 252.73 99.06 0)
