File: dispEncoder.kicad_sch (KiCad schematic)
At the start: 14 parts, among them SW1 RotaryEncoder_Switch_MP, U9 74AHC595

Commit message: Almost done
Schematic done
PCB missing ground planes
Need Coopilot review
Parts:
- R300: renamed from RV1; footprint Potentiometer_THT:Potentiometer_Piher_PT-10-V05_Vertical -> Potentiometer_THT:Potentiometer_Bourns_3339P_Vertical_HandSoldering
- renumbered C2 to C300, C10 to C310, C7 to C311, C5 to C312, DS1 to DS300, R39 to R310, R32 to R311, R29 to R312, R41 to R313, R27 to R314, R23 to R315, SW1 to SW310, U9 to U300
Changed lines of the file:
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@@
 		)
 	)
-	(global_label "SDA{slash}SDI"
-		(shape bidirectional)
-		(at 215.9 107.95 0)
-		(fields_autoplaced yes)
+	(hierarchical_label "SDO"
+		(shape input)
+		(at 187.96 85.09 180)
 		(effects
 			(font
 				(size 1.27 1.27)
 			)
-			(justify left)
-		)
-		(property "Intersheetrefs" "${INTERSHEET_REFS}"
-			(at 227.9794 107.95 0)
-			(effects
-				(font
-					(size 1.27 1.27)
-				)
-				(justify left)
-				(hide yes)
-			)
-		)
-	)
-	(global_label "DISP"
-		(shape bidirectional)
+			(justify right)
+		)
+	)
+	(hierarchical_label "DISP"
+		(shape input)
 		(at 187.96 97.79 180)
-		(fields_autoplaced yes)
 		(effects
 			(font
@@
 			(justify right)
 		)
-		(property "Intersheetrefs" "${INTERSHEET_REFS}"
-			(at 179.5092 97.79 0)
-			(effects
-				(font
-					(size 1.27 1.27)
-				)
-				(justify right)
-				(hide yes)
-			)
-		)
-	)
-	(global_label "SWS"
-		(shape bidirectional)
-		(at 134.62 83.82 0)
-		(fields_autoplaced yes)
+	)
+	(hierarchical_label "SCL"
+		(shape input)
+		(at 187.96 90.17 180)
 		(effects
 			(font
 				(size 1.27 1.27)
 			)
-			(justify left)
-		)
-		(property "Intersheetrefs" "${INTERSHEET_REFS}"
-			(at 142.5869 83.82 0)
-			(effects
-				(font
-					(size 1.27 1.27)
-				)
-				(justify left)
-				(hide yes)
-			)
-		)
-	)
-	(global_label "SWA"
-		(shape bidirectional)
-		(at 48.26 83.82 180)
-		(fields_autoplaced yes)
+			(justify right)
+		)
+	)
+	(hierarchical_label "SDA{slash}SDI"
+		(shape output)
+		(at 215.9 107.95 0)
 		(effects
 			(font
 				(size 1.27 1.27)
 			)
-			(justify right)
-		)
-		(property "Intersheetrefs" "${INTERSHEET_REFS}"
-			(at 40.414 83.82 0)
-			(effects
-				(font
-					(size 1.27 1.27)
-				)
-				(justify right)
-				(hide yes)
-			)
-		)
-	)
-	(global_label "SDO"
-		(shape bidirectional)
-		(at 187.96 85.09 180)
-		(fields_autoplaced yes)
+			(justify left)
+		)
+	)
+	(hierarchical_label "SWB"
+		(shape output)
+		(at 48.26 93.98 180)
 		(effects
 			(font
@@
 			(justify right)
 		)
-		(property "Intersheetrefs" "${INTERSHEET_REFS}"
-			(at 180.0535 85.09 0)
-			(effects
-				(font
-					(size 1.27 1.27)
-				)
-				(justify right)
-				(hide yes)
-			)
-		)
-	)
-	(global_label "SCL"
-		(shape bidirectional)
-		(at 187.96 90.17 180)
-		(fields_autoplaced yes)
+	)
+	(hierarchical_label "SWA"
+		(shape output)
+		(at 48.26 83.82 180)
 		(effects
 			(font
@@
 			(justify right)
 		)
-		(property "Intersheetrefs" "${INTERSHEET_REFS}"
-			(at 180.3559 90.17 0)
-			(effects
-				(font
-					(size 1.27 1.27)
-				)
-				(justify right)
-				(hide yes)
-			)
-		)
-	)
-	(global_label "SWB"
-		(shape bidirectional)
-		(at 48.26 93.98 180)
-		(fields_autoplaced yes)
+	)
+	(hierarchical_label "SWS"
+		(shape output)
+		(at 134.62 83.82 0)
 		(effects
 			(font
 				(size 1.27 1.27)
 			)
-			(justify right)
-		)
-		(property "Intersheetrefs" "${INTERSHEET_REFS}"
-			(at 40.2326 93.98 0)
-			(effects
-				(font
-					(size 1.27 1.27)
-				)
-				(justify right)
-				(hide yes)
-			)
+			(justify left)
 		)
 	)
@@
 		(dnp no)
 		(fields_autoplaced yes)
-		(property "Reference" "C7"
+		(property "Reference" "C311"
 			(at 69.85 99.0599 0)
 			(effects
@@
 			(project "Motor Control"
 				(path "/287fa568-d091-4161-b3b2-3036dfbfe9fa/8050a139-abb0-4450-a33e-db857d70c5ca"
-					(reference "C7")
+					(reference "C311")
 					(unit 1)
 				)
@@
 		(dnp no)
 		(fields_autoplaced yes)
-		(property "Reference" "DS1"
-			(at 246.0341 54.61 0)
+		(property "Reference" "DS300"
+			(at 245.9833 54.61 0)
 			(effects
 				(font
@@
 		)
 		(property "Value" "WC1602A"
-			(at 246.0341 57.15 0)
+			(at 245.9833 57.15 0)
 			(effects
 				(font
@@
 			(project "Motor Control"
 				(path "/287fa568-d091-4161-b3b2-3036dfbfe9fa/8050a139-abb0-4450-a33e-db857d70c5ca"
-					(reference "DS1")
+					(reference "DS300")
 					(unit 1)
 				)
@@
 		(dnp no)
 		(fields_autoplaced yes)
-		(property "Reference" "R39"
+		(property "Reference" "R310"
 			(at 116.84 76.1999 0)
 			(effects
@@
 			(project "Motor Control"
 				(path "/287fa568-d091-4161-b3b2-3036dfbfe9fa/8050a139-abb0-4450-a33e-db857d70c5ca"
-					(reference "R39")
+					(reference "R310")
 					(unit 1)
 				)
@@
 		(dnp no)
 		(fields_autoplaced yes)
-		(property "Reference" "U9"
-			(at 205.3941 77.47 0)
+		(property "Reference" "U300"
+			(at 205.3433 77.47 0)
 			(effects
 				(font
@@
 		)
 		(property "Value" "74AHC595"
-			(at 205.3941 80.01 0)
+			(at 205.3433 80.01 0)
 			(effects
 				(font
@@
 			(project "Motor Control"
 				(path "/287fa568-d091-4161-b3b2-3036dfbfe9fa/8050a139-abb0-4450-a33e-db857d70c5ca"
-					(reference "U9")
+					(reference "U300")
 					(unit 1)
 				)
@@
 		(dnp no)
 		(fields_autoplaced yes)
-		(property "Reference" "R32"
+		(property "Reference" "R311"
 			(at 86.36 76.1999 0)
 			(effects
@@
 			(project "Motor Control"
 				(path "/287fa568-d091-4161-b3b2-3036dfbfe9fa/8050a139-abb0-4450-a33e-db857d70c5ca"
-					(reference "R32")
+					(reference "R311")
 					(unit 1)
 				)
@@
 		(on_board yes)
 		(dnp no)
-		(property "Reference" "SW1"
+		(property "Reference" "SW310"
 			(at 106.68 80.01 0)
 			(effects
@@
 			(project "Motor Control"
 				(path "/287fa568-d091-4161-b3b2-3036dfbfe9fa/8050a139-abb0-4450-a33e-db857d70c5ca"
-					(reference "SW1")
+					(reference "SW310")
 					(unit 1)
 				)
@@
 		(dnp no)
 		(fields_autoplaced yes)
-		(property "Reference" "C10"
+		(property "Reference" "C310"
 			(at 134.62 99.0599 0)
 			(effects
@@
 			(project "Motor Control"
 				(path "/287fa568-d091-4161-b3b2-3036dfbfe9fa/8050a139-abb0-4450-a33e-db857d70c5ca"
-					(reference "C10")
+					(reference "C310")
 					(unit 1)
 				)
@@
 		(dnp no)
 		(fields_autoplaced yes)
-		(property "Reference" "R29"
+		(property "Reference" "R312"
 			(at 77.47 76.1999 0)
 			(effects
@@
 			(project "Motor Control"
 				(path "/287fa568-d091-4161-b3b2-3036dfbfe9fa/8050a139-abb0-4450-a33e-db857d70c5ca"
-					(reference "R29")
+					(reference "R312")
 					(unit 1)
 				)
@@
 		(on_board yes)
 		(dnp no)
-		(property "Reference" "C2"
+		(property "Reference" "C300"
 			(at 194.31 69.8499 0)
 			(effects
@@
 			(project "Motor Control"
 				(path "/287fa568-d091-4161-b3b2-3036dfbfe9fa/8050a139-abb0-4450-a33e-db857d70c5ca"
-					(reference "C2")
+					(reference "C300")
 					(unit 1)
 				)
@@
 		(dnp no)
 		(fields_autoplaced yes)
-		(property "Reference" "RV1"
+		(property "Reference" "R300"
 			(at 262.89 60.9599 0)
 			(effects
@@
 			)
 		)
-		(property "Footprint" "Potentiometer_THT:Potentiometer_Piher_PT-10-V05_Vertical"
+		(property "Footprint" "Potentiometer_THT:Potentiometer_Bourns_3339P_Vertical_HandSoldering"
 			(at 260.35 62.23 0)
 			(effects
@@
 			(project "Motor Control"
 				(path "/287fa568-d091-4161-b3b2-3036dfbfe9fa/8050a139-abb0-4450-a33e-db857d70c5ca"
-					(reference "RV1")
+					(reference "R300")
 					(unit 1)
 				)
@@
 		(dnp no)
 		(fields_autoplaced yes)
-		(property "Reference" "C5"
+		(property "Reference" "C312"
 			(at 57.15 99.0599 0)
 			(effects
@@
 			(project "Motor Control"
 				(path "/287fa568-d091-4161-b3b2-3036dfbfe9fa/8050a139-abb0-4450-a33e-db857d70c5ca"
-					(reference "C5")
+					(reference "C312")
 					(unit 1)
 				)
@@
 		(dnp no)
 		(fields_autoplaced yes)
-		(property "Reference" "R23"
+		(property "Reference" "R315"
 			(at 58.42 88.9 90)
 			(effects
@@
 			(project "Motor Control"
 				(path "/287fa568-d091-4161-b3b2-3036dfbfe9fa/8050a139-abb0-4450-a33e-db857d70c5ca"
-					(reference "R23")
+					(reference "R315")
 					(unit 1)
 				)
@@
 		(dnp no)
 		(fields_autoplaced yes)
-		(property "Reference" "R27"
+		(property "Reference" "R314"
 			(at 71.12 78.74 90)
 			(effects
@@
 			(project "Motor Control"
 				(path "/287fa568-d091-4161-b3b2-3036dfbfe9fa/8050a139-abb0-4450-a33e-db857d70c5ca"
-					(reference "R27")
+					(reference "R314")
 					(unit 1)
 				)
@@
 		(dnp no)
 		(fields_autoplaced yes)
-		(property "Reference" "R41"
+		(property "Reference" "R313"
 			(at 125.73 78.74 90)
 			(effects
@@
 			(project "Motor Control"
 				(path "/287fa568-d091-4161-b3b2-3036dfbfe9fa/8050a139-abb0-4450-a33e-db857d70c5ca"
-					(reference "R41")
-					(unit 1)
-				)
+					(reference "R313")
+					(unit 1)
+				)

Commit message: V 1.0 fabrication output
V 1.0 ready for fabrication
Other:
- company: (none) -> AARHUS TECH
- title: (none) -> Motor Control
Changed lines of the file:
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@@
 	(generator_version "9.0")
 	(paper "A4")
+	(title_block
+		(title "Motor Control")
+		(rev "1.0")
+		(company "AARHUS TECH")
+	)
 	(junction
 		(at 130.81 83.82)

Commit message: Partnumbers
Parts:
- U300: Part number (none) -> 100-0763; Supplier (none) -> RS

Commit message: BOM
Parts:
- C300, C310, C311, C312: Part number (none) -> 135-8304; Supplier (none) -> RS
- DS300: Part number (none) -> 1218634; Supplier (none) -> Farnell
- R300: value 50k -> 20k; Part number (none) -> 167-3259; Supplier (none) -> RS
- R310, R311, R312: Part number (none) -> 05.000.0510; Supplier (none) -> Cypax
- R313, R314, R315: Part number (none) -> 05.000.0410; Supplier (none) -> Cypax
- SW310: Part number (none) -> 781-6830; Supplier (none) -> RS
Changed lines of the file:
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@@
 			)
 		)
-		(property "Part number" ""
+		(property "Part number" "135-8304"
 			(at 66.04 100.33 0)
 			(effects
@@
 			)
 		)
-		(property "Supplier" ""
+		(property "Supplier" "RS"
 			(at 66.04 100.33 0)
 			(effects
@@
 			)
 		)
-		(property "Part number" ""
+		(property "Part number" "1218634"
 			(at 243.84 77.47 0)
 			(effects
@@
 			)
 		)
-		(property "Supplier" ""
+		(property "Supplier" "Farnell"
 			(at 243.84 77.47 0)
 			(effects
@@
 			)
 		)
-		(property "Part number" ""
+		(property "Part number" "05.000.0510 "
 			(at 119.38 77.47 0)
 			(effects
@@
 			)
 		)
-		(property "Supplier" ""
+		(property "Supplier" "Cypax"
 			(at 119.38 77.47 0)
 			(effects
@@
 			)
 		)
-		(property "Part number" ""
+		(property "Part number" "05.000.0510 "
 			(at 88.9 77.47 0)
 			(effects
@@
 			)
 		)
-		(property "Supplier" ""
+		(property "Supplier" "Cypax"
 			(at 88.9 77.47 0)
 			(effects
@@
 			)
 		)
-		(property "Part number" ""
+		(property "Part number" "781-6830"
 			(at 106.68 86.36 0)
 			(effects
@@
 			)
 		)
-		(property "Supplier" ""
+		(property "Supplier" "RS"
 			(at 106.68 86.36 0)
 			(effects
@@
 			)
 		)
-		(property "Part number" ""
+		(property "Part number" "135-8304"
 			(at 130.81 100.33 0)
 			(effects
@@
 			)
 		)
-		(property "Supplier" ""
+		(property "Supplier" "RS"
 			(at 130.81 100.33 0)
 			(effects
@@
 			)
 		)
-		(property "Part number" ""
+		(property "Part number" "05.000.0510 "
 			(at 80.01 77.47 0)
 			(effects
@@
 			)
 		)
-		(property "Supplier" ""
+		(property "Supplier" "Cypax"
 			(at 80.01 77.47 0)
 			(effects
@@
 			)
 		)
-		(property "Part number" ""
+		(property "Part number" "135-8304"
 			(at 198.12 71.12 0)
 			(effects
@@
 			)
 		)
-		(property "Supplier" ""
+		(property "Supplier" "RS"
 			(at 198.12 71.12 0)
 			(effects
@@
 			)
 		)
-		(property "Value" "50k"
+		(property "Value" "20k"
 			(at 262.89 63.4999 0)
 			(effects
@@
 			)
 		)
-		(property "Part number" ""
+		(property "Part number" "167-3259"
 			(at 260.35 62.23 0)
 			(effects
@@
 			)
 		)
-		(property "Supplier" ""
+		(property "Supplier" "RS"
 			(at 260.35 62.23 0)
 			(effects
@@
 			)
 		)
-		(property "Part number" ""
+		(property "Part number" "135-8304"
 			(at 53.34 100.33 0)
 			(effects
@@
 			)
 		)
-		(property "Supplier" ""
+		(property "Supplier" "RS"
 			(at 53.34 100.33 0)
 			(effects
@@
 			)
 		)
-		(property "Part number" ""
+		(property "Part number" "05.000.0410 "
 			(at 58.42 93.98 90)
 			(effects
@@
 			)
 		)
-		(property "Supplier" ""
+		(property "Supplier" "Cypax"
 			(at 58.42 93.98 90)
 			(effects
@@
 			)
 		)
-		(property "Part number" ""
+		(property "Part number" "05.000.0410 "
 			(at 71.12 83.82 90)
 			(effects
@@
 			)
 		)
-		(property "Supplier" ""
+		(property "Supplier" "Cypax"
 			(at 71.12 83.82 90)
 			(effects
@@
 			)
 		)
-		(property "Part number" ""
+		(property "Part number" "05.000.0410 "
 			(at 125.73 83.82 90)
 			(effects
@@
 			)
 		)
-		(property "Supplier" ""
+		(property "Supplier" "Cypax"
 			(at 125.73 83.82 90)
 			(effects

Commit message: V 2.0
Parts:
- added R300: 10k, Resistor_THT:R_Axial_DIN0207_L6.3mm_D2.5mm_P10.16mm_Horizontal, symbol Device:R
- renumbered R300 to R301
Connections:
- net +5V: now also R300.2
- net GNDD: no longer U300.10 (~{SRCLR})
- net at U300.15 (QA): no longer DS300.11 (D4)
- net at U300.1 (QB): no longer DS300.12 (D5)
- net D6_{disp}: now reaches DS300.13 (D6)
- net D6_{disp}: now also U300.6 (QG); no longer U300.2 (QC)
- net D7_{disp}: now reaches DS300.14 (D7)
- net D7_{disp}: now also U300.7 (QH); no longer U300.3 (QD)
- net D5_{disp}: now reaches U300.5 (QF)
- net D5_{disp}: now also DS300.12 (D5); no longer DS300.4 (RS)
- net E_{disp}: now reaches DS300.6 (E)
- net E_{disp}: now also U300.3 (QD); no longer U300.7 (QH)
- net D4_{disp}: now reaches U300.4 (QE)
- net D4_{disp}: now also DS300.11 (D4)
- net DISP renamed DISP_{SS}
- net SCL renamed SCL/PGC
- net SDA/SDI: no longer names the net of U300.9 (QH')
- net SDO renamed MOSI/PGD
- new net: R300.1, U300.10 (~{SRCLR})
- new net RS_{disp}: DS300.4 (RS), U300.2 (QC)
- no-connect marks 4 -> 5
